File: payload_carrier.kicad_pcb (KiCad board)
At the start: 2 copper layers, 46 parts, among them J1 Conn_01x02, J2 USB_C_Receptacle_USB2.0_16P, J3 Conn_01x08, J4 Conn_01x08, J5 Conn_01x05, J6 Micro_SD_Card, SW1 SW_MEC_5G, U1 TPS73733DCQR, U2 TPS562242DRLR, U3 STM32G0B1CBTx, Y1 Crystal

Commit message: done
Parts:
- removed SW1: SW_MEC_5G, Button_Switch_SMD:SW_MEC_5GSH9
- added G***: LOGO, LOGO, F.Cu at (130.6, 58.4)
- added G***: LOGO, LOGO, F.Cu at (145.7, 78.8)
- added G***: LOGO, LOGO, B.Cu at (125.5, 55.8)
- added H1: MountingHole, Mounting_Wuerth:Mounting_Wuerth_WA-SMSI-M3_H0.5mm_9774005360, F.Cu at (106.9, 35.0)
- added H2: MountingHole, Mounting_Wuerth:Mounting_Wuerth_WA-SMSI-M3_H0.5mm_9774005360, F.Cu at (144.8, 35.0)
- added H4: MountingHole, Mounting_Wuerth:Mounting_Wuerth_WA-SMSI-M3_H0.5mm_9774005360, F.Cu at (106.9, 57.0)
- added SW2: SW_MEC_5E, Button_Switch_SMD:SW_SPST_B3SL-1002P, F.Cu at (144.0, 43.8)
- moved C6 122.4 mm to (142.1, 76.0), turned to 180 degrees
- moved J1 118.6 mm to (137.5, 77.9), turned to 180 degrees
- moved C7 116.1 mm to (139.3, 68.5), turned to 90 degrees
- moved C9 114.8 mm to (139.8, 65.3), turned to -90 degrees
- moved J4 113.4 mm to (137.2, 40.6)
- moved D1 113.0 mm to (133.5, 65.6)
- moved R4 112.4 mm to (138.8, 71.8)
- moved R3 110.9 mm to (135.8, 71.8)
- moved C16 110.8 mm to (135.8, 73.3)
- moved R1 109.8 mm to (137.0, 70.0)
- moved R2 108.5 mm to (137.0, 68.4), turned to 180 degrees
- moved Y1 104.4 mm to (124.4, 36.9)
- moved C10 103.3 mm to (133.1, 38.8), turned to 90 degrees
- moved J5 102.5 mm to (142.0, 60.1), turned to 180 degrees
- moved R5 102.4 mm to (129.8, 69.7), turned to 180 degrees
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Connections:
- net /USB_DM renamed /USB_D-
- net /USB_DP renamed /USB_D+
- U3 pad 18: unconnected-(U3-PA7-Pad18) -> /MB_MOSI
Routing:
- net +5V: track 0.00 -> 58.0 mm, vias 0 -> 4
- net /NRST: track 0.00 -> 44.2 mm, vias 0 -> 1
- net /SD_CS: track 0.00 -> 40.7 mm
- net /SD_MOSI: track 0.00 -> 29.7 mm, vias 0 -> 2
- net /SD_CLK: track 0.00 -> 29.5 mm, vias 0 -> 2
- net /SD_MISO: track 0.00 -> 27.4 mm
- net /USB_D+: track 0.00 -> 27.2 mm
- net +3.3V: track 0.00 -> 26.5 mm, vias 0 -> 12
- net /USB_D-: track 0.00 -> 25.1 mm
- net GND: track 0.00 -> 22.3 mm, vias 0 -> 53
- net Net-(D1-A): track 0.00 -> 20.0 mm
- net /SWDIO: track 0.00 -> 19.3 mm
- net /SWDCLK: track 0.00 -> 16.9 mm, vias 0 -> 1
- net /MB_SDA: track 0.00 -> 16.9 mm
- net /MB_INT: track 0.00 -> 14.0 mm, vias 0 -> 1
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- added copper zone on In2.Cu, net +3.3V
- added copper zone on B.Cu, net GND
- added copper zone on F.Cu, net GND
- added copper zone on In1.Cu, net GND
Other:
- board outline added: 47.9 x 50.8 mm
- copper layers 2 -> 4
- board text added: "+"
- board text added: "-"
- board text added: "3v"
- board text added: "3v3"
- board text added: "5v"
- board text added: "gnd"
- board text added: "nrst"
- board text added: "tortilla"
- board text added: "v0.1"
- board text added: "wclk"
- board text added: "wdio"
