File: payload_carrier.kicad_sch (KiCad schematic)
At the start: 46 parts, among them J1 Conn_01x02, J2 USB_C_Receptacle_USB2.0_16P, J3 Conn_01x08, J4 Conn_01x08, J5 Conn_01x05, J6 Micro_SD_Card, SW1 SW_MEC_5G, U1 TPS73733DCQR, U2 TPS562242DRLR, U3 STM32G0B1CBTx, Y1 Crystal

Commit message: PCB Layout Prelim Changes
Parts:
- C10: footprint (none) -> Capacitor_SMD:C_0603_1608Metric
- R11: footprint (none) -> Resistor_SMD:R_0603_1608Metric
- U2: footprint (none) -> Package_TO_SOT_SMD:SOT-563
Connections:
- net MB_MOSI: no longer U3.18 (PA7)

Commit message: done
Parts:
- removed SW1: SW_MEC_5G, Button_Switch_SMD:SW_MEC_5GSH9, symbol KiCad:SW_MEC_5G
- added H1, H2, H3, H4: MountingHole, Mounting_Wuerth:Mounting_Wuerth_WA-SMSI-M3_H0.5mm_9774005360, symbol Mechanical:MountingHole
- added SW2: SW_MEC_5E, Button_Switch_SMD:SW_SPST_B3SL-1002P, symbol Switch:SW_MEC_5E
Connections:
- net GND: now also SW2.2, SW2.3 (K)
- net MB_MOSI: now also U3.18 (PA7)
- net NRST: now also SW2.1
- net USB_DM renamed USB_D-
- net USB_DP renamed USB_D+
